Commit message: Fised wheel rotation direction and image processing

File: src/my_robot/urdf/my_robot.xacro (robot description, xacro)
@@ -170,5 +170,5 @@
     <child link="right_wheel"/>
     <parent link="chassis"/>
-    <axis xyz="0 -1 0" rpy="0 0 0"/>
+    <axis xyz="0 1 0" rpy="0 0 0"/>
     <limit effort="10000" velocity="1000"/>
     <dynamics damping="1.0" friction="1.0"/>

Commit message: Initial commit

File: src/my_robot/urdf/my_robot.xacro (robot description, xacro)
@@ -125,4 +125,11 @@
     </collision>
   </link>
+  <joint name="camera_optical_joint" type="fixed">
+    <origin xyz="0 0 0" rpy="-1.5707 0 -1.5707"/>
+    <parent link="camera"/>
+    <child link="camera_link_optical"/>
+  </joint>
+  <link name="camera_link_optical">
+  </link>
   <link name='hokuyo'>
     <inertial>
@@ -156,5 +163,5 @@
     <child link="hokuyo"/>
     <parent link="chassis"/>
-    <axis xyz="0 1 0" rpy="0 0 0"/>
+    <axis xyz="0 0 0" rpy="0 0 0"/>
   </joint>
   <joint type="continuous" name="left_wheel_hinge">
